File: solo/USB-nano.brd (EAGLE design)
At the start: 13 x 10.6 mm, 19 parts, among them U1 USB_TRACES_NANO

Commit message: update button outline
Parts:
- removed S2: TOUCH_SENSOR, efm-fido:SOMU_CAPACITIVE_TOUCH_PAD
- moved S1 18.8 mm to (30.0, 20.0), turned to 180 degrees
Connections:
- net N$5: now also S1.P$2, S1.SENSE2; no longer S2.P$1, S2.SENSE
Routing:
- net N$5: track 10.2 -> 11.1 mm
Changed lines of the file:
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@@
 <drawing>
 <settings>
-<setting alwaysvectorfont="yes"/>
+<setting alwaysvectorfont="no"/>
 <setting verticaltext="up"/>
 </settings>
@@
 <layer number="28" name="bValues" color="7" fill="1" visible="yes" active="yes"/>
 <layer number="29" name="tStop" color="7" fill="3" visible="no" active="yes"/>
-<layer number="30" name="bStop" color="7" fill="6" visible="no" active="yes"/>
+<layer number="30" name="bStop" color="7" fill="6" visible="yes" active="yes"/>
 <layer number="31" name="tCream" color="7" fill="4" visible="no" active="yes"/>
 <layer number="32" name="bCream" color="7" fill="5" visible="no" active="yes"/>
@@
 <layer number="38" name="bTest" color="7" fill="1" visible="no" active="yes"/>
 <layer number="39" name="tKeepout" color="4" fill="11" visible="yes" active="yes"/>
-<layer number="40" name="bKeepout" color="1" fill="11" visible="no" active="yes"/>
+<layer number="40" name="bKeepout" color="1" fill="11" visible="yes" active="yes"/>
 <layer number="41" name="tRestrict" color="4" fill="10" visible="yes" active="yes"/>
-<layer number="42" name="bRestrict" color="1" fill="10" visible="no" active="yes"/>
+<layer number="42" name="bRestrict" color="1" fill="10" visible="yes" active="yes"/>
 <layer number="43" name="vRestrict" color="2" fill="10" visible="yes" active="yes"/>
 <layer number="44" name="Drills" color="7" fill="1" visible="no" active="yes"/>
@@
 <wire x1="9.474609375" y1="10.67963125" x2="9.474609375" y2="20.140459375" width="0.1" layer="49"/>
 <text x="2.65" y="19.95" size="0.6096" layer="26" font="vector" ratio="16" rot="MR0">v0.1</text>
+<rectangle x1="9.9" y1="20" x2="10.15" y2="21.05" layer="42"/>
+<rectangle x1="9.9" y1="9.7" x2="10.3" y2="11.05" layer="42"/>
 </plain>
 <attributes>
@@
 <attribute name="VALUE" x="7.318" y="21.875" size="1.27" layer="27" rot="R180" display="off"/>
 </element>
-<element name="S1" library="efm-fido" library_urn="urn:adsk.eagle:library:4245354" package="SOMU_CAPACITIVE_TOUCH_PAD" package3d_urn="urn:adsk.eagle:package:10401338/2" value="TOUCH_SENSOR" x="11.22" y="18.62" smashed="yes"/>
 <element name="R2" library="efm-fido" library_urn="urn:adsk.eagle:library:4245354" package="R0402" package3d_urn="urn:adsk.eagle:package:4245807/8" value="1k 1%" x="4.72" y="11.68" smashed="yes" rot="MR90">
 <attribute name="NAME" x="6.305" y="10.765" size="0.6096" layer="26" ratio="15" rot="MR0"/>
@@
 <attribute name="VALUE" x="1.455" y="13.405" size="1.27" layer="28" rot="MR180" display="off"/>
 </element>
-<element name="S2" library="efm-fido" library_urn="urn:adsk.eagle:library:4245354" package="SOMU_CAPACITIVE_TOUCH_PAD" package3d_urn="urn:adsk.eagle:package:10401338/2" value="TOUCH_SENSOR" x="11.23" y="12.42" smashed="yes"/>
 <element name="R3" library="efm-fido" library_urn="urn:adsk.eagle:library:4245354" package="R0402" package3d_urn="urn:adsk.eagle:package:4245807/8" value="1k 1%" x="3.9" y="11.68" smashed="yes" rot="MR90">
 <attribute name="NAME" x="3.435" y="10.415" size="0.6096" layer="26" ratio="15" rot="MR0"/>
 <attribute name="VALUE" x="1.995" y="11.045" size="1.27" layer="28" rot="MR90" display="off"/>
 </element>
+<element name="S1" library="efm-fido" library_urn="urn:adsk.eagle:library:4245354" package="SOMU_CAPACITIVE_TOUCH_PAD" package3d_urn="urn:adsk.eagle:package:10401338/5" value="TOUCH_SENSOR" x="30" y="20" smashed="yes" rot="R180"/>
 </elements>
 <signals>
@@
 </signal>
 <signal name="N$2">
-<contactref element="S1" pad="P$1"/>
-<contactref element="S1" pad="SENSE"/>
 <contactref element="R2" pad="1"/>
 <wire x1="4.72" y1="11.055" x2="4.9172375" y2="11.055" width="0.1524" layer="16"/>
@@
 <wire x1="8.0571" y1="10.8192" x2="9.9712" y2="12.7333" width="0.1524" layer="16"/>
 <wire x1="9.9712" y1="12.7333" x2="9.9712" y2="16.6512" width="0.1524" layer="16"/>
-<wire x1="9.9712" y1="16.6512" x2="11.1" y2="17.78" width="0.1524" layer="16"/>
-<wire x1="11.1" y1="17.78" x2="11.1" y2="18.13" width="0.1524" layer="16"/>
-<wire x1="12.22" y1="18.62" x2="11.2146375" y2="18.135" width="0.1524" layer="16"/>
-<wire x1="11.2146375" y1="18.135" x2="11.1" y2="18.60095" width="0.1524" layer="16"/>
-<wire x1="12.22" y1="18.62" x2="12.22" y2="18.62" width="0" layer="19" extent="1-16"/>
-<wire x1="11.1" y1="18.13" x2="11.2146375" y2="18.135" width="0" layer="19" extent="16-16"/>
+<contactref element="S1" pad="P$1"/>
+<contactref element="S1" pad="SENSE"/>
+<wire x1="11.103146875" y1="18.20956875" x2="11.1059875" y2="18.206728125" width="0.1524" layer="16"/>
+<wire x1="10.39278125" y1="17.07278125" x2="10.39278125" y2="17.811346875" width="0.1524" layer="16"/>
+<wire x1="10.39278125" y1="17.811346875" x2="10.791003125" y2="18.20956875" width="0.1524" layer="16"/>
+<wire x1="10.791003125" y1="18.20956875" x2="11.103146875" y2="18.20956875" width="0.1524" layer="16"/>
+<wire x1="11.1059875" y1="18.206728125" x2="11.357540625" y2="18.206728125" width="0.1524" layer="16"/>
+<wire x1="11.357540625" y1="18.206728125" x2="11.772815625" y2="17.791453125" width="0.1524" layer="16"/>
+<wire x1="11.772815625" y1="17.791453125" x2="11.772815625" y2="17.4715875" width="0.1524" layer="16"/>
+<wire x1="9.9712" y1="16.6512" x2="10.39278125" y2="17.07278125" width="0.1524" layer="16"/>
+<wire x1="11.437" y1="16.878" x2="11.437" y2="16.878" width="0" layer="19" extent="1-16"/>
+<wire x1="11.772815625" y1="17.4715875" x2="11.437" y2="16.878" width="0" layer="19" extent="16-16"/>
 </signal>
 <signal name="N$4">
@@
 </signal>
 <signal name="N$5">
-<contactref element="S2" pad="P$1"/>
-<contactref element="S2" pad="SENSE"/>
 <contactref element="R3" pad="1"/>
 <wire x1="3.9" y1="11.055" x2="3.91855" y2="11.055" width="0.1524" layer="16"/>
@@
 <wire x1="10.65810625" y1="13.106609375" x2="10.8" y2="13.33" width="0.1524" layer="16"/>
 <wire x1="10.8" y1="13.33" x2="10.8" y2="13.0841375" width="0.1524" layer="16"/>
-<wire x1="8.1852" y1="10.5652" x2="10.65810625" y2="13.03810625" width="0.1524" layer="16"/>
+<wire x1="8.1852" y1="10.5652" x2="10.185" y2="12.565" width="0.1524" layer="16"/>
+<wire x1="10.4651625" y1="12.8451625" x2="10.65810625" y2="13.03810625" width="0.1524" layer="16"/>
 <wire x1="10.65810625" y1="13.03810625" x2="10.65810625" y2="13.106609375" width="0.1524" layer="16"/>
-<wire x1="12.23" y1="12.42" x2="11.73" y2="12.6008" width="0.1524" layer="16"/>
-<wire x1="11.73" y1="12.6008" x2="11.45" y2="11.73" width="0.1524" layer="16"/>
-<wire x1="12.23" y1="12.42" x2="12.23" y2="12.42" width="0" layer="19" extent="1-16"/>
-<wire x1="10.8" y1="13.0841375" x2="11.73" y2="12.6008" width="0" layer="19" extent="16-16"/>
+<contactref element="S1" pad="SENSE2"/>
+<contactref element="S1" pad="P$2"/>
+<wire x1="11.597046875" y1="13.087509375" x2="11.597046875" y2="13.0943375" width="0.1524" layer="16"/>
+<wire x1="11.3547" y1="12.8451625" x2="11.597046875" y2="13.087509375" width="0.1524" layer="16"/>
+<wire x1="10.185" y1="12.565" x2="10.4651625" y2="12.8451625" width="0.1524" layer="16"/>
+<wire x1="10.4651625" y1="12.8451625" x2="11.3547" y2="12.8451625" width="0.1524" layer="16"/>
+<wire x1="11.597046875" y1="13.0943375" x2="11.5283" y2="13.163084375" width="0.1524" layer="16"/>
+<wire x1="11.5283" y1="13.163084375" x2="11.5283" y2="14.0707" width="0.1524" layer="16"/>
+<wire x1="11.5283" y1="14.0707" x2="11.448" y2="14.151" width="0.1524" layer="16"/>
+<wire x1="11.448" y1="14.151" x2="11.448" y2="14.151" width="0" layer="19" extent="1-16"/>
 </signal>
 <signal name="N$6">

Commit message: Update USB-nano.brd
Parts:
- moved C3 0.80 mm to (1.27, 12.3)
- moved C1 0.20 mm to (1.89, 11.5)
- moved R2 0.10 mm to (4.82, 11.7)
- moved SWDIO 0.05 mm to (5.99, 12.3)
