File: kicad/solo-A/solo-A.kicad_pcb (KiCad board)
At the start: 2 copper layers, 28 x 15 mm, 18 parts, among them T1 TLV742p, U1 LPC55S28JEV98K

Commit message: kicad solo2 progress
Parts:
- added Z1: BZA900A, Package_TO_SOT_SMD:SOT-665, F.Cu at (120.8, 48.5)
- moved C10 10.4 mm to (128.8, 57.2), turned to 270 degrees
- moved C8 10.1 mm to (128.1, 57.2), turned to 270 degrees
- moved C6 9.87 mm to (127.2, 57.2), turned to 270 degrees
- moved C4 9.66 mm to (126.5, 57.2), turned to 270 degrees
- moved C2 9.57 mm to (125.7, 57.2), turned to 270 degrees
- moved D1 8.73 mm to (132.9, 50.5), turned to 270 degrees
- moved T1 8.17 mm to (123.1, 57.1)
- moved C11 8.11 mm to (120.9, 57.1)
- moved C12 8.01 mm to (121.7, 57.1)
- moved U1 3.68 mm to (125.7, 52.5)
- moved D2 2.10 mm to (120.7, 52.2), turned to 180 degrees
- moved C1 1.54 mm to (123.5, 47.9)
- moved N1 1.53 mm to (141.4, 48.4)
- moved C3 1.48 mm to (124.3, 47.8)
- moved C7 1.48 mm to (126.0, 47.8)
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Routing:
- net +3V3: track 65.0 -> 74.8 mm, vias 9 -> 13
- net /solo/5V: track 3.42 -> 12.5 mm
- net GNDREF: track 67.9 -> 74.9 mm, vias 3 -> 1
- net /solo/Sheet5DDC9C58/SPI_MISO: track 9.08 -> 15.3 mm
- net /solo/Sheet5DDC9C58/SWCLK: track 4.82 -> 10.8 mm
- net /solo/Sheet5DDC9C58/SPI_SS: track 8.17 -> 14.1 mm
- net /solo/Sheet5DDC9C58/SPI_CLK: track 9.13 -> 14.6 mm
- net /solo/Sheet5DDC9C58/SPI_MOSI: track 8.69 -> 14.2 mm
- net /solo/D-: track 0.00 -> 3.47 mm
- net /solo/Sheet5DDC9C58/SWO: track 6.36 -> 9.35 mm, vias 1 -> 3
- net Net-(D2-Pad4): track 5.31 -> 2.47 mm
- net /solo/Sheet5DDC9C58/B: track 5.17 -> 2.34 mm
- net /solo/D+: track 0.00 -> 2.69 mm
- net /solo/Sheet5DDC9C58/G: track 0.00 -> 2.55 mm
- net /solo/nRESET: track 12.1 -> 13.8 mm, vias 3 -> 1
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Other:
- board size 28 x 15 mm -> 45.8 x 15 mm
- board text added: "Place imports at abs(100,100) Cover outline at Eco1"
- board text removed: "Place imports at abs(100,100)"
