File: kicad/solo-A/solo.sch (KiCad schematic (older format))
At the start: 18 parts, among them T1 TLV742p

Commit message: kicad solo2 progress
Parts:
- added Z1: BZA900A, Package_TO_SOT_SMD:SOT-665, symbol solo:BZA900A
Connections:
- wire segments 122 -> 130
- no-connect marks 1 -> 2
Changed lines of the file:
@@
 	-1   0    0    1
 $EndComp
+$Comp
+L solo:BZA900A Z1
+U 1 1 5DFCBD03
+P 7750 5150
+F 0 "Z1" H 7750 5265 50  0000 C CNN
+F 1 "BZA900A" H 7750 5174 50  0000 C CNN
+F 2 "Package_TO_SOT_SMD:SOT-665" H 7450 5150 50  0001 C CNN
+F 3 "" H 7450 5150 50  0001 C CNN
+	1    7750 5150
+	1    0    0    -1
+$EndComp
+Text Label 7100 5300 0    50   ~ 0
+D+
+Text Label 7100 5400 0    50   ~ 0
+D-
+Wire Wire Line
+	7100 5300 7500 5300
+Wire Wire Line
+	7100 5400 7350 5400
+Wire Wire Line
+	7350 5400 7350 5450
+Wire Wire Line
+	7350 5450 7500 5450
+Wire Wire Line
+	7150 5550 7400 5550
+Wire Wire Line
+	7400 5550 7400 5600
+Wire Wire Line
+	7400 5600 7500 5600
+NoConn ~ 7500 5750
+Text Label 7150 5550 0    50   ~ 0
+5V
+$Comp
+L power:GNDREF #PWR?
+U 1 1 5E0181F2
+P 8250 5500
+F 0 "#PWR?" H 8250 5250 50  0001 C CNN
+F 1 "GNDREF" V 8255 5372 50  0000 R CNN
+F 2 "" H 8250 5500 50  0001 C CNN
+F 3 "" H 8250 5500 50  0001 C CNN
+	1    8250 5500
+	0    -1   -1   0
+$EndComp
+Wire Wire Line
+	8250 5500 8000 5500
 $EndSCHEMATC
