File: kicad/solo-C.sch (KiCad schematic (older format))
At the start: 8 parts, among them P1 USB_C_Plug

Commit message: add plating
Parts:
- P1: Description (none) -> USB-C plug connector; MPN (none) -> 632712000112; Manufacturer (none) -> Wurth Electronics; Package (none) -> Custom, USB-C plug; Pins (none) -> 26
Changed lines of the file:
@@
 F 2 "solo:USB-C_WURTH" H 2250 3700 50  0001 C CNN
 F 3 "https://www.usb.org/sites/default/files/documents/usb_type-c.zip" H 2250 3700 50  0001 C CNN
+F 4 "Wurth Electronics" H 2100 3700 50  0001 C CNN "Manufacturer"
+F 5 "USB-C plug connector" H 2100 3700 50  0001 C CNN "Description"
+F 6 "632712000112" H 2100 3700 50  0001 C CNN "MPN"
+F 7 "26" H 2100 3700 50  0001 C CNN "Pins"
+F 8 "Custom, USB-C plug" H 2100 3700 50  0001 C CNN "Package"
 	1    2100 3700
 	1    0    0    -1
